Commit message: Add materials to visual elements in URDF

File: p2/catkin_ws/src/my_robot/urdf/my_robot.xacro (robot description, xacro)
@@ -28,4 +28,7 @@
         <box size=".4 .2 .1"/>
       </geometry>
+      <material name="blue">
+        <color rgba="0 0 1 1"/>
+      </material>
     </visual>
     <!-- Casters -->
@@ -75,4 +78,7 @@
         <cylinder radius="0.1" length="0.05"/>
       </geometry>
+      <material name="black">
+        <color rgba="0 0 0 1"/>
+      </material>
     </visual>
   </link>
@@ -97,4 +103,7 @@
         <cylinder radius="0.1" length="0.05"/>
       </geometry>
+      <material name="black">
+        <color rgba="0 0 0 1"/>
+      </material>
     </visual>
   </link>
@@ -137,4 +146,7 @@
         <box size="0.05 0.05 0.05"/>
       </geometry>
+      <material name="red">
+        <color rgba="1 0 0 1"/>
+      </material>
     </visual>
   </link>
@@ -165,4 +177,7 @@
         <mesh filename="package://my_robot/meshes/hokuyo.dae"/>
       </geometry>
+      <material name="black">
+        <color rgba="0 0 0 1"/>
+      </material>
     </visual>
   </link>

Commit message: Remove material definitions from my_robot.xacro
Removed material definitions for various visual elements in the URDF.

File: p2/catkin_ws/src/my_robot/urdf/my_robot.xacro (robot description, xacro)
@@ -28,7 +28,4 @@
         <box size=".4 .2 .1"/>
       </geometry>
-      <material name="blue">
-        <color rgba="0 0 1 1"/>
-      </material>
     </visual>
     <!-- Casters -->
@@ -78,7 +75,4 @@
         <cylinder radius="0.1" length="0.05"/>
       </geometry>
-      <material name="black">
-        <color rgba="0 0 0 1"/>
-      </material>
     </visual>
   </link>
@@ -103,7 +97,4 @@
         <cylinder radius="0.1" length="0.05"/>
       </geometry>
-      <material name="black">
-        <color rgba="0 0 0 1"/>
-      </material>
     </visual>
   </link>
@@ -146,7 +137,4 @@
         <box size="0.05 0.05 0.05"/>
       </geometry>
-      <material name="red">
-        <color rgba="1 0 0 1"/>
-      </material>
     </visual>
   </link>
@@ -177,7 +165,4 @@
         <mesh filename="package://my_robot/meshes/hokuyo.dae"/>
       </geometry>
-      <material name="black">
-        <color rgba="0 0 0 1"/>
-      </material>
     </visual>
   </link>
